Commit message: Makes panda use the generic environment.

File: optuna_fabrics/tune/panda.urdf (robot description, URDF)
Before this commit: robot panda, 14 links, 13 joints
Links:
- removed link panda_leftfinger
- removed link panda_rightfinger
- added link panda_link5_offset, mass 1.00
- link panda_hand: mass 0.68 -> 1.00; geometry visual sphere radius=0.01
- link panda_link0: geometry collision mesh filename=meshes/panda/collision/link0.stl; visual mesh filename=meshes/panda/visual/link0.obj
- link panda_link1: geometry collision mesh filename=meshes/panda/collision/link1.stl; visual mesh filename=meshes/panda/visual/link1.obj
- link panda_link2: geometry collision mesh filename=meshes/panda/collision/link2.stl; visual mesh filename=meshes/panda/visual/link2.obj
- link panda_link3: geometry collision mesh filename=meshes/panda/collision/link3.stl; visual mesh filename=meshes/panda/visual/link3.obj
- link panda_link4: geometry collision mesh filename=meshes/panda/collision/link4.stl; visual mesh filename=meshes/panda/visual/link4.obj
- link panda_link5: geometry collision mesh filename=meshes/panda/collision/link5.stl; visual mesh filename=meshes/panda/visual/link5.obj
- link panda_link6: geometry collision mesh filename=meshes/panda/collision/link6.stl; visual mesh filename=meshes/panda/visual/link6.obj
- link panda_link7: geometry collision mesh filename=meshes/panda/collision/link7.stl; visual mesh filename=meshes/panda/visual/link7.obj
Joints:
- removed joint panda_finger_joint1
- removed joint panda_finger_joint2
- added joint panda_joint5_offset: type fixed, parent panda_link5, child panda_link5_offset, origin xyz=0 0 -0.20 rpy=0 0 0

Commit message: Genericify the examples.

File: optuna_fabrics/tune/panda.urdf (robot description, URDF)
Before this commit: robot panda, 13 links, 12 joints
Links:
- link world: mass None -> 1000
